File: kiboard_wireless.kicad_sch (KiCad schematic)
At the start: 117 parts, among them J1 USB_C_Receptacle_USB2.0_16P, J2 Conn_01x02_Shielded, J3 TC2030_SWD, Q1 2N7002, SW1 SW_Nidec_CAS-120A1, SW2 SW_Push_45deg, U1 nRF52840_E73-2G4M08S1C, U2 WE-TVS-824015043, U3 BQ24075RGT, U4 MAX17048

Commit message: pain
Connections:
- net +BATT: no longer D2.1 (K), R4.2
- net scl: now also U1.10 (P0.30/AIN6)
- net sda: now also U1.9 (P0.31/AIN7)
- new net: D2.1 (K), R4.2
Other:
- moved on the sheet: D2, R4
Changed lines of the file:
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@@
   (junction (at 228.6 27.94) (diameter 0) (color 0 0 0 0)
   )
-  (junction (at 242.57 107.95) (diameter 0) (color 0 0 0 0)
-  )
   (junction (at 54.61 175.26) (diameter 0) (color 0 0 0 0)
   )
@@
   (junction (at 85.09 175.26) (diameter 0) (color 0 0 0 0)
   )
+  (junction (at 245.11 107.95) (diameter 0) (color 0 0 0 0)
+  )
   (junction (at 31.75 158.75) (diameter 0) (color 0 0 0 0)
   )
   (junction (at 54.61 142.24) (diameter 0) (color 0 0 0 0)
   )
-  (junction (at 242.57 115.57) (diameter 0) (color 0 0 0 0)
-  )
   (junction (at 92.71 142.24) (diameter 0) (color 0 0 0 0)
   )
@@
     (stroke (width 0) (type default))
   )
-  (wire (pts (xy 242.57 107.95) (xy 261.62 107.95))
-    (stroke (width 0) (type default))
-  )
   (wire (pts (xy 229.87 161.29) (xy 224.79 161.29))
     (stroke (width 0) (type default))
@@
     (stroke (width 0) (type default))
   )
-  (wire (pts (xy 237.49 107.95) (xy 242.57 107.95))
+  (wire (pts (xy 237.49 107.95) (xy 245.11 107.95))
     (stroke (width 0) (type default))
   )
@@
     (stroke (width 0) (type default))
   )
+  (wire (pts (xy 245.11 106.68) (xy 245.11 107.95))
+    (stroke (width 0) (type default))
+  )
   (wire (pts (xy 39.37 158.75) (xy 39.37 175.26))
     (stroke (width 0) (type default))
@@
     (stroke (width 0) (type default))
   )
+  (wire (pts (xy 245.11 114.3) (xy 245.11 118.11))
+    (stroke (width 0) (type default))
+  )
   (wire (pts (xy 201.93 166.37) (xy 207.01 166.37))
     (stroke (width 0) (type default))
@@
     (stroke (width 0) (type default))
   )
-  (wire (pts (xy 242.57 115.57) (xy 242.57 118.11))
-    (stroke (width 0) (type default))
-  )
   (wire (pts (xy 85.09 175.26) (xy 85.09 191.77))
     (stroke (width 0) (type default))
@@
     (stroke (width 0) (type default))
   )
+  (wire (pts (xy 86.36 60.96) (xy 85.09 60.96))
+    (stroke (width 0) (type default))
+  )
   (wire (pts (xy 213.36 67.31) (xy 212.09 67.31))
     (stroke (width 0) (type default))
@@
     (stroke (width 0) (type default))
   )
-  (wire (pts (xy 242.57 115.57) (xy 254 115.57))
+  (wire (pts (xy 237.49 115.57) (xy 254 115.57))
     (stroke (width 0) (type default))
   )
@@
     (stroke (width 0) (type default))
   )
+  (wire (pts (xy 86.36 58.42) (xy 85.09 58.42))
+    (stroke (width 0) (type default))
+  )
   (wire (pts (xy 77.47 137.16) (xy 77.47 142.24))
     (stroke (width 0) (type default))
@@
     (stroke (width 0) (type default))
   )
-  (wire (pts (xy 237.49 115.57) (xy 242.57 115.57))
-    (stroke (width 0) (type default))
-  )
   (wire (pts (xy 97.79 154.94) (xy 105.41 154.94))
     (stroke (width 0) (type default))
@@
     (stroke (width 0) (type default))
   )
-  (wire (pts (xy 237.49 128.27) (xy 242.57 128.27))
+  (wire (pts (xy 237.49 128.27) (xy 245.11 128.27))
     (stroke (width 0) (type default))
   )
@@
     (stroke (width 0) (type default))
   )
-  (wire (pts (xy 242.57 128.27) (xy 242.57 123.19))
+  (wire (pts (xy 245.11 128.27) (xy 245.11 123.19))
     (stroke (width 0) (type default))
   )
@@
     (stroke (width 0) (type default))
   )
+  (wire (pts (xy 245.11 107.95) (xy 261.62 107.95))
+    (stroke (width 0) (type default))
+  )
   (wire (pts (xy 254 115.57) (xy 254 118.11))
     (stroke (width 0) (type default))
@@
     )
   )
+  (global_label "scl" (shape bidirectional) (at 86.36 58.42 0) (fields_autoplaced)
+    (effects (font (size 1.27 1.27)) (justify left))
+    (property "Intersheetrefs" "${INTERSHEET_REFS}" (at 93.2384 58.42 0)
+      (effects (font (size 1.27 1.27)) (justify left) hide)
+    )
+  )
   (global_label "usb-D+" (shape input) (at 267.97 63.5 0) (fields_autoplaced)
     (effects (font (size 1.27 1.27)) (justify left))
@@
     )
   )
+  (global_label "sda" (shape bidirectional) (at 86.36 60.96 0) (fields_autoplaced)
+    (effects (font (size 1.27 1.27)) (justify left))
+    (property "Intersheetrefs" "${INTERSHEET_REFS}" (at 93.7826 60.96 0)
+      (effects (font (size 1.27 1.27)) (justify left) hide)
+    )
+  )
   (global_label "SWCLK" (shape input) (at 39.37 43.18 180) (fields_autoplaced)
     (effects (font (size 1.27 1.27)) (justify right))
@@
     )
   )
-  (symbol (lib_id "Device:LED") (at 242.57 111.76 90) (unit 1)
+  (symbol (lib_id "Device:LED") (at 245.11 110.49 90) (unit 1)
     (in_bom yes) (on_board yes) (dnp no)
-    (property "Reference" "D2" (at 241.3 102.87 90)
+    (property "Reference" "D2" (at 243.84 101.6 90)
       (effects (font (size 1.27 1.27)) (justify right))
     )
-    (property "Value" "LED" (at 241.3 105.41 90)
+    (property "Value" "LED" (at 243.84 104.14 90)
       (effects (font (size 1.27 1.27)) (justify right))
     )
-    (property "Footprint" "LED_SMD:LED_1206_3216Metric" (at 242.57 111.76 0)
+    (property "Footprint" "LED_SMD:LED_1206_3216Metric" (at 245.11 110.49 0)
       (effects (font (size 1.27 1.27)) hide)
     )
-    (property "Datasheet" "~" (at 242.57 111.76 0)
+    (property "Datasheet" "~" (at 245.11 110.49 0)
       (effects (font (size 1.27 1.27)) hide)
     )
@@
     )
   )
-  (symbol (lib_id "Device:R_Small") (at 242.57 120.65 180) (unit 1)
+  (symbol (lib_id "Device:R_Small") (at 245.11 120.65 180) (unit 1)
     (in_bom yes) (on_board yes) (dnp no)
-    (property "Reference" "R4" (at 246.38 119.38 0)
+    (property "Reference" "R4" (at 248.92 119.38 0)
       (effects (font (size 1.27 1.27)) (justify left))
     )
-    (property "Value" "1.5 kOhm" (at 252.73 121.92 0)
+    (property "Value" "1.5 kOhm" (at 255.27 121.92 0)
       (effects (font (size 1.27 1.27)) (justify left))
     )
-    (property "Footprint" "Resistor_SMD:R_1206_3216Metric" (at 242.57 120.65 0)
+    (property "Footprint" "Resistor_SMD:R_1206_3216Metric" (at 245.11 120.65 0)
       (effects (font (size 1.27 1.27)) hide)
     )
-    (property "Datasheet" "~" (at 242.57 120.65 0)
+    (property "Datasheet" "~" (at 245.11 120.65 0)
       (effects (font (size 1.27 1.27)) hide)
     )

Commit message: done
Parts:
- removed U2: WE-TVS-824015043, Package_TO_SOT_SMD:SOT-23-6, symbol Power_Protection:WE-TVS-824015043
- added U5: SRV05-4, PCM_marbastlib-various:SOT-23-6-routable, symbol PCM_marbastlib-various:SRV05-4
Connections:
- net VSENSE is gone; now on net col05: U1.7 (P0.02/AIN0)
- net +5V: now also U5.5 (VP)
- net GND: now also U5.2 (VN)
- net col00: now also U1.11 (P0.00/XL1)
- net col01: now also U1.13 (P0.01/XL2)
- net col02: now also U1.15 (P0.05/AIN3)
- net col03: now also U1.4 (P0.28/AIN4)
- net col04: now also U1.6 (P1.13)
- net col06: now also U1.1 (P1.11)
- net col07: now also U1.2 (P1.10)
- net col08: now also U1.3 (P0.03/AIN1)
- net col09: now also U1.17 (P1.09)
- net col10: now also U1.33 (P0.13)
- net col11: now also U1.35 (P0.24)
- net row0: now also U1.8 (P0.29/AIN5)
- net usb-D+: now also U5.4 (IO3)
- net usb-D-: now also U5.1 (IO1)
