File: kiboard_wireless.kicad_pcb (KiCad board)
At the start: 2 copper layers, 237 x 98.8 mm, 117 parts, among them J1 USB_C_Receptacle_USB2.0_16P, J2 Conn_01x02_Shielded, J3 TC2030_SWD, Q1 2N7002, SW1 SW_Nidec_CAS-120A1, SW2 SW_Push_45deg, U1 nRF52840_E73-2G4M08S1C, U2 WE-TVS-824015043, U3 BQ24075RGT, U4 MAX17048

Commit message: keymatrix done
Routing:
- net (no net): track 0.00 -> 382.5 mm
- net row3: track 0.00 -> 209.5 mm
- net row1: track 0.00 -> 209.5 mm
- net row2: track 0.00 -> 209.5 mm
- net row0: track 0.00 -> 95.2 mm
- net col08: track 0.00 -> 71.4 mm
- net col07: track 0.00 -> 71.4 mm
- net col06: track 0.00 -> 71.4 mm
- net col05: track 0.00 -> 71.4 mm
- net col04: track 0.00 -> 71.4 mm
- net col03: track 0.00 -> 71.4 mm
- net col11: track 0.00 -> 38.1 mm
- net col10: track 0.00 -> 38.1 mm
- net col09: track 0.00 -> 38.1 mm
- net col02: track 0.00 -> 38.1 mm
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
Commit message: fixed weird trace
Routing:
- net (no net): track 382.5 -> 0.00 mm
Changed lines of the file:
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@@
   (gr_line (start 36.25 107.25) (end 32.25 107.25)
     (stroke (width 0.1) (type default)) (layer "Edge.Cuts"))
-  (segment (start 166.22619 111.375) (end 265.301776 111.375) (width 0.25) (layer "B.Cu") (net 0))
-  (segment (start 156 111.375) (end 166.22619 111.375) (width 0.25) (layer "B.Cu") (net 0))
-  (segment (start 265.301776 111.375) (end 284.5 92.176776) (width 0.25) (layer "B.Cu") (net 0))
-  (segment (start 166.22619 111.375) (end 182 111.375) (width 0.25) (layer "B.Cu") (net 0))
-  (segment (start 156 114.5) (end 156 111.375) (width 0.25) (layer "B.Cu") (net 0))
-  (segment (start 225 111.375) (end 147.17619 111.375) (width 0.25) (layer "B.Cu") (net 0))
-  (segment (start 284.5 92.176776) (end 284.5 2.25) (width 0.25) (layer "B.Cu") (net 0))
-  (segment (start 265.301776 111.375) (end 225 111.375) (width 0.25) (layer "B.Cu") (net 0))
-  (segment (start 166.22619 111.375) (end 147.17619 111.375) (width 0.25) (layer "B.Cu") (net 0))
   (segment (start 147.17619 20.9) (end 128.12619 20.9) (width 0.25) (layer "B.Cu") (net 67))
   (segment (start 166.22619 20.9) (end 147.17619 20.9) (width 0.25) (layer "B.Cu") (net 67))

Commit message: pain
Parts:
- moved J3 367.8 mm to (260.2, 88.6), turned to 0 degrees
- moved SW2 349.2 mm to (255.5, 78.5)
- moved U1 347.9 mm to (257.7, 98.2), turned to 90 degrees
- moved R12 300.2 mm to (244.8, 103.5), turned to 90 degrees
- moved R13 298.0 mm to (242.2, 103.5), turned to 90 degrees
- moved U4 287.8 mm to (239.4, 103.3), turned to 0 degrees
- moved C5 279.3 mm to (235.8, 102.9)
- moved R1 167.2 mm to (45.2, 88.8)
- moved R2 167.2 mm to (42.8, 88.8)
- moved D1 167.0 mm to (49.1, 87.5)
- moved J1 167.0 mm to (38.6, 85.0)
- moved L2 167.0 mm to (49.1, 90.0)
- moved F1 146.9 mm to (14.8, 69.8), turned to 90 degrees
- moved L1 145.6 mm to (18.5, 69.2)
- moved U2 145.3 mm to (51.0, 84.2), turned to 90 degrees
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Connections:
- D2 pad 1: +BATT -> Net-(D2-K)
- R4 pad 2: +BATT -> Net-(D2-K)
- U1 pad 10: unconnected-(U1-P0.30/AIN6-Pad10) -> scl
- U1 pad 9: unconnected-(U1-P0.31/AIN7-Pad9) -> sda
Routing:
- net +3.3V: track 0.00 -> 36.4 mm, vias 0 -> 2
- net GND: track 0.00 -> 24.3 mm
- net usb-D-: track 0.00 -> 21.5 mm, vias 0 -> 2
- net usb-D+: track 0.00 -> 19.2 mm, vias 0 -> 2
- net GNDPWR: track 0.00 -> 17.9 mm, vias 0 -> 2
- net +BATT: track 0.00 -> 17.0 mm
- net VBUS: track 0.00 -> 15.4 mm, vias 0 -> 2
- net sda: track 0.00 -> 14.0 mm
- net scl: track 0.00 -> 11.8 mm
- net RST: track 0.00 -> 11.6 mm
- net Net-(J1-CC2): track 0.00 -> 8.70 mm, vias 0 -> 2
- net Net-(Q1-G): track 0.00 -> 5.78 mm
- net Earth: track 0.00 -> 5.16 mm
- net +VSW: track 0.00 -> 5.03 mm
- net Net-(D2-K): track 0.00 -> 3.43 mm
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
Commit message: done
Parts:
- removed U2: WE-TVS-824015043, Package_TO_SOT_SMD:SOT-23-6
- added U5: SRV05-4, PCM_marbastlib-various:SOT-23-6-routable, B.Cu at (48.6, 84.4)
- moved Q1 178.7 mm to (82.3, 102.8), turned to -90 degrees
- moved R10 175.8 mm to (82.0, 99.2), turned to 0 degrees
- moved R9 172.0 mm to (78.5, 103.2), turned to 90 degrees
- moved SW1 154.1 mm to (67.4, 109.2), turned to 0 degrees
- moved R11 138.7 mm to (62.9, 100.3), turned to 90 degrees
- moved R7 137.9 mm to (76.6, 95.5), turned to 180 degrees
- moved C4 137.7 mm to (76.6, 98.0), turned to 0 degrees
- moved R4 137.0 mm to (75.9, 89.5), turned to 90 degrees
- moved D2 132.3 mm to (73.1, 89.4), turned to -90 degrees
- moved R6 130.1 mm to (73.4, 101.6), turned to 90 degrees
- moved U3 128.8 mm to (71.9, 94.2), turned to 0 degrees
- moved C2 127.5 mm to (70.6, 89.2), turned to 90 degrees
- moved C3 122.5 mm to (68.1, 89.2), turned to 90 degrees
- moved R8 121.8 mm to (68.6, 97.7), turned to 0 degrees
- moved R5 119.6 mm to (67.4, 95.2), turned to 0 degrees
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Connections:
- U1 pad 1: unconnected-(U1-P1.11-Pad1) -> col06
- U1 pad 11: unconnected-(U1-P0.00/XL1-Pad11) -> col00
- U1 pad 13: unconnected-(U1-P0.01/XL2-Pad13) -> col01
- U1 pad 15: unconnected-(U1-P0.05/AIN3-Pad15) -> col02
- U1 pad 17: unconnected-(U1-P1.09-Pad17) -> col09
- U1 pad 2: unconnected-(U1-P1.10-Pad2) -> col07
- U1 pad 3: unconnected-(U1-P0.03/AIN1-Pad3) -> col08
- U1 pad 33: unconnected-(U1-P0.13-Pad33) -> col10
- U1 pad 35: unconnected-(U1-P0.24-Pad35) -> col11
- U1 pad 4: unconnected-(U1-P0.28/AIN4-Pad4) -> col03
- U1 pad 6: unconnected-(U1-P1.13-Pad6) -> col04
- U1 pad 7: VSENSE -> col05
- U1 pad 8: unconnected-(U1-P0.29/AIN5-Pad8) -> row0
Routing:
- net GND: track 24.3 -> 345.7 mm, vias 0 -> 10
- net +5V: track 3.37 -> 232.6 mm, vias 0 -> 8
- net col00: track 38.1 -> 259.7 mm, vias 0 -> 3
- net +BATT: track 17.0 -> 230.1 mm, vias 0 -> 2
- net usb-D+: track 19.2 -> 228.7 mm
- net usb-D-: track 21.5 -> 227.3 mm
- net col01: track 38.1 -> 239.8 mm, vias 0 -> 3
- net col02: track 38.1 -> 221.0 mm, vias 0 -> 3
- net col03: track 71.4 -> 236.5 mm, vias 0 -> 1
- net col04: track 71.4 -> 214.4 mm, vias 0 -> 1
- net col05: track 71.4 -> 193.6 mm, vias 0 -> 1
- net col06: track 71.4 -> 183.2 mm
- net col07: track 71.4 -> 162.3 mm
- net col08: track 71.4 -> 141.5 mm
- net row0: track 95.2 -> 152.5 mm, vias 0 -> 2
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Other:
- board size 237 x 98.8 mm -> 237.1 x 98.8 mm

Commit message: improvements
Routing:
- net usb-D+: track 228.7 -> 225.8 mm
- net usb-D-: track 227.3 -> 225.4 mm

Commit message: bump
Routing:
- net GND: track 345.7 -> 5.81 mm, vias 10 -> 0
- net usb-D-: track 225.4 -> 220.5 mm, vias 2 -> 0
- net usb-D+: track 225.8 -> 222.5 mm, vias 2 -> 0
- net +BATT: track 230.1 -> 232.4 mm, vias 2 -> 3
- net +5V: track 232.6 -> 233.8 mm
- net col02: track 221.0 -> 220.7 mm, vias 3 -> 2
- net col00: track 259.7 -> 259.4 mm, vias 3 -> 2
- net row0: track 152.5 -> 152.7 mm, vias 2 -> 0
- net col09: vias 3 -> 1
- net col01: vias 3 -> 2
- added copper zone on B.Cu, net GND
